Commit message: feat: add whole body urdf and mujoco xml file for T1

File: resources/T1/T1_serial.urdf (robot description, URDF)
Before this commit: robot T1, 24 links, 23 joints
Links:
- link AL1: geometry visual mesh filename=meshes/AL1.STL
- link AL2: geometry visual mesh filename=meshes/AL2.STL
- link AL3: geometry collision cylinder length=0.15 radius=0.03; visual mesh filename=meshes/AL3.STL
- link AR1: geometry visual mesh filename=meshes/AR1.STL
- link AR2: geometry visual mesh filename=meshes/AR2.STL
- link AR3: geometry collision cylinder length=0.15 radius=0.03; visual mesh filename=meshes/AR3.STL
- link Hip_Roll_Left: geometry visual mesh filename=meshes/Hip_Roll_Left.STL
- link Hip_Roll_Right: geometry visual mesh filename=meshes/Hip_Roll_Right.STL
- link Hip_Yaw_Left: geometry collision cylinder length=0.16 radius=0.05; visual mesh filename=meshes/Hip_Yaw_Left.STL
- link Hip_Yaw_Right: geometry collision cylinder length=0.16 radius=0.05; visual mesh filename=meshes/Hip_Yaw_Right.STL
- link Shank_Left: geometry collision cylinder length=0.15 radius=0.05; visual mesh filename=meshes/Shank_Left.STL
- link Shank_Right: geometry collision cylinder length=0.15 radius=0.05; visual mesh filename=meshes/Shank_Right.STL
- link left_hand_link: geometry collision cylinder length=0.175 radius=0.03; visual mesh filename=meshes/left_hand_link.STL
- link right_hand_link: geometry collision cylinder length=0.175 radius=0.03; visual mesh filename=meshes/right_hand_link.STL
Joints:
- joint Left_Ankle_Pitch: limit lower=-0.87 upper=0.35 effort=12 velocity=18.8 -> lower=-0.87 upper=0.35 effort=20 velocity=18.8
- joint Left_Ankle_Roll: limit lower=-0.44 upper=0.44 effort=12 velocity=12.4 -> lower=-0.44 upper=0.44 effort=15 velocity=12.4
- joint Left_Hip_Roll: limit lower=-0.52 upper=1.57 effort=45 velocity=10.9 -> lower=-0.2 upper=1.57 effort=30 velocity=10.9
- joint Left_Knee_Pitch: limit lower=0 upper=2.34 effort=65 velocity=11.7 -> lower=0 upper=2.34 effort=60 velocity=11.7
- joint Right_Ankle_Pitch: limit lower=-0.87 upper=0.35 effort=12 velocity=18.8 -> lower=-0.87 upper=0.35 effort=20 velocity=18.8
- joint Right_Ankle_Roll: limit lower=-0.44 upper=0.44 effort=12 velocity=12.4 -> lower=-0.44 upper=0.44 effort=15 velocity=12.4
- joint Right_Hip_Roll: limit lower=-1.57 upper=0.52 effort=30 velocity=10.9 -> lower=-1.57 upper=0.2 effort=30 velocity=10.9
- joint Right_Knee_Pitch: limit lower=0 upper=2.34 effort=65 velocity=11.7 -> lower=0 upper=2.34 effort=60 velocity=11.7
